Commit message: Laser plugin added

File: custom_robot/description/robot.urdf.xacro (robot description, xacro)
@@ -5,3 +5,4 @@
     <xacro:include filename="robot_core.xacro" />
     <xacro:include filename="g_control.xacro"/>
+    <xacro:include filename="lidar.xacro"/>
 </robot>

File: custom_robot/description/robot_core.xacro (robot description, xacro)
@@ -45,7 +45,6 @@
         </xacro:inertial_box>
     </link>
-    <!-- <xacro:gazebo_material link_name="chassis_link" color="yellow"/> -->
     <gazebo reference="chassis_link">
-        <material>gazebo/yellow</material>
+        <material>Gazebo/Yellow</material>
     </gazebo>
     <!--LEFT WHEEL LINK-->
@@ -69,7 +68,6 @@
     </link>
     <gazebo reference="left_wheel">
-        <material>gazebo/black</material>
+        <material>Gazebo/Black</material>
     </gazebo>
-    <!-- <xacro:gazebo_material link_name="left_wheel" color="black"/> -->
     <joint name="left_wheel_joint" type="continuous">
         <origin xyz="0 0.175 0" rpy="0 0 0"/>
@@ -97,7 +95,6 @@
         </xacro:inertial_cylinder>
     </link>
-    <!-- <xacro:gazebo_material link_name="right_wheel" color="black"/> -->
     <gazebo reference="right_wheel">
-        <material>gazebo/black</material>
+        <material>Gazebo/Black</material>
     </gazebo>
     <joint name="right_wheel_joint" type="continuous">
@@ -126,7 +123,6 @@
         </xacro:inertial_sphere>
     </link>
-    <!-- <xacro:gazebo_material link_name="caster_wheel" color="black"/>  -->
     <gazebo reference="caster_wheel">
-        <material>gazebo/black</material>
+        <material>Gazebo/Black</material>
         <mu1 value="0.001"/>
         <mu2 value="0.001"/>

Commit message: remove comments

File: custom_robot/description/robot.urdf.xacro (robot description, xacro)
@@ -1,6 +1,4 @@
 <?xml version="1.0"?>
 <robot xmlns:xacro="http://www.ros.org/wiki/xacro"  name="robot">
-    <!-- Example link -->
-    <!-- <link name="base_link"></link> -->
     <xacro:include filename="robot_core.xacro" />
     <xacro:include filename="g_control.xacro"/>
