Commit message: wheel rotation adjusted

File: custom_robot/description/robot_core.xacro (robot description, xacro)
@@ -52,5 +52,5 @@
     <link name="left_wheel">
         <visual>
-            <origin xyz="0 0.0 0" rpy="0 0 0"/>
+            <origin xyz="0 0.0 0" rpy="${pi/2} 0 0"/>
             <geometry>
                 <cylinder radius="0.06" length="0.04"/>
@@ -59,5 +59,5 @@
         </visual>
         <collision>
-            <origin xyz="0 0.0 0" rpy="0 0 0"/>
+            <origin xyz="0 0.0 0" rpy="${pi/2} 0 0"/>
             <geometry>
                 <cylinder radius="0.06" length="0.04"/>
@@ -73,13 +73,13 @@
     <!-- <xacro:gazebo_material link_name="left_wheel" color="black"/> -->
     <joint name="left_wheel_joint" type="continuous">
-        <origin xyz="0 0.175 0" rpy="-${pi/2} 0 0"/>
+        <origin xyz="0 0.175 0" rpy="0 0 0"/>
         <parent link="base_link"/>
         <child link="left_wheel"/>
-        <axis xyz="0 0 1"/>
+        <axis xyz="0 1 0"/>
     </joint>
     <!--RIGHT WHEEL LINK-->
     <link name="right_wheel">
         <visual>
-            <origin xyz="0 -0.0 0" rpy="0 0 0"/>
+            <origin xyz="0 0.0 0" rpy="${pi/2} 0 0"/>
             <geometry>
                 <cylinder radius="0.06" length="0.04"/>
@@ -88,5 +88,5 @@
         </visual>
         <collision>
-            <origin xyz="0 -0.0 0" rpy="0 0 0"/>
+            <origin xyz="0 0.0 0" rpy="${pi/2} 0 0"/>
             <geometry>
                 <cylinder radius="0.06" length="0.04"/>
@@ -94,5 +94,5 @@
         </collision>
         <xacro:inertial_cylinder mass="0.1" length="0.04" radius="0.06">
-            <origin xyz="0 -0.0 0" rpy="0 0 0" />
+            <origin xyz="0 0.0 0" rpy="0 0 0" />
         </xacro:inertial_cylinder>
     </link>
@@ -102,8 +102,8 @@
     </gazebo>
     <joint name="right_wheel_joint" type="continuous">
-        <origin xyz="0 -0.175 0" rpy="${pi/2} 0 0"/>
+        <origin xyz="0 -0.175 0" rpy="0 0 0"/>
         <parent link="base_link"/>
         <child link="right_wheel"/>
-        <axis xyz="0 0 1"/>
+        <axis xyz="0 1 0"/>
     </joint>
     <!--CASTER WHEEL LINK-->

Commit message: added basefootprint link under base_link

File: custom_robot/description/robot_core.xacro (robot description, xacro)
@@ -21,4 +21,12 @@
     <!--BASE_LINK-->
     <link name="base_link"> </link>
+    <!--BASE_FOOTPRINT LINK-->
+    <link name="base_footprint"></link>
+    <joint name="base_footprint_joint" type="fixed">
+        <origin xyz="0 0 0" rpy="0 0 0"/>
+        <parent link="base_link"/>
+        <child link="base_footprint"/>
+    </joint>
+    <!--CHASSIS_LINK-->
     <joint name="chassis_joint" type="fixed">
         <origin xyz="-0.1 0 0" rpy="0 0 0"/>
@@ -26,5 +34,4 @@
         <child link="chassis_link"/>
     </joint>
-    <!--CHASSIS_LINK-->
     <link name="chassis_link">
         <visual>
