Commit message: increase samples and pitch adjustment

File: custom_robot/description/lidar.xacro (robot description, xacro)
@@ -4,5 +4,5 @@
         <parent link="chassis_link"/>
         <child link="laser_frame"/>
-        <origin xyz="0.1 0 0.175" rpy="0 0 0"/>
+        <origin xyz="0.1 0 0.175" rpy="0 -0.07 0"/>
     </joint>
     <link name="laser_frame">
@@ -32,7 +32,8 @@
                 <scan>
                     <horizontal>
-                        <samples>360</samples>
-                        <min_angle>-3.14</min_angle>
-                        <max_angle>3.14</max_angle>
+                        <samples>720</samples>
+                        <resolution>1</resolution>
+                        <min_angle>-3.141592</min_angle>
+                        <max_angle>3.141592</max_angle>
                     </horizontal>
                 </scan>
@@ -40,4 +41,5 @@
                     <min>0.3</min>
                     <max>12</max>
+                    <resolution>1</resolution>
                 </range>
             </ray>

Commit message: camera added

File: custom_robot/description/lidar.xacro (robot description, xacro)
@@ -27,5 +27,5 @@
         <sensor name="laser" type="ray">
             <pose> 0 0 0 0 0 0 </pose>
-            <visualize>true</visualize>
+            <visualize>false</visualize>
             <update_rate>10</update_rate>
             <ray>

File: custom_robot/description/robot.urdf.xacro (robot description, xacro)
@@ -1,6 +1,7 @@
 <?xml version="1.0"?>
 <robot xmlns:xacro="http://www.ros.org/wiki/xacro"  name="robot">
-    <xacro:include filename="robot_core.xacro" />
+    <xacro:include filename="robot_core.xacro"/>
     <xacro:include filename="g_control.xacro"/>
     <xacro:include filename="lidar.xacro"/>
+    <xacro:include filename="camera.xacro"/>
 </robot>

File: custom_robot/description/robot_core.xacro (robot description, xacro)
@@ -22,5 +22,5 @@
     <link name="base_link"> </link>
     <!--BASE_FOOTPRINT LINK-->
-    <link name="base_footprint"></link>
+    <link name="base_footprint"> </link>
     <joint name="base_footprint_joint" type="fixed">
         <origin xyz="0 0 0" rpy="0 0 0"/>
